File: pcb/ram.sch (KiCad schematic (older format))
At the start: 12 parts, among them J1 CONN_INTEGRALSTICK_FPGA_DEVICE, U2 XC7A50T-1FTG256C, U3 S27KS0641, U4 S27KS0641

Commit message: Initial routing of LVCMOS18 GPIO bus. Hooked up a few 0603 decoupling caps.
Connections:
- net GPIO_1V8_10: now also U2.H4 (IO_L18N_T2_35); no longer U2.J5 (IO_L19P_T3_35)
- net GPIO_1V8_14: now also U2.J4 (IO_L19N_T3_VREF_35); no longer U2.L2 (IO_L23N_T3_35)
- net GPIO_1V8_15: now also U2.L2 (IO_L23N_T3_35); no longer U2.H4 (IO_L18N_T2_35)
- net GPIO_1V8_16: now also U2.H5 (IO_L18P_T2_35); no longer U2.K2 (IO_L24N_T3_35)
- net GPIO_1V8_17: now also U2.J5 (IO_L19P_T3_35); no longer U2.K5 (IO_25_35)
- net GPIO_1V8_6: now also U2.E5 (IO_L13N_T2_MRCC_35); no longer U2.J4 (IO_L19N_T3_VREF_35)
- net GPIO_1V8_7: now also U2.K2 (IO_L24N_T3_35); no longer U2.E6 (IO_0_35)
- net GPIO_1V8_8: now also U2.E6 (IO_0_35); no longer U2.H5 (IO_L18P_T2_35)
- net GPIO_1V8_9: now also U2.K5 (IO_25_35); no longer U2.E5 (IO_L13N_T2_MRCC_35)
Changed lines of the file:
@@
 Text Label 8600 5100 2    50   ~ 0
 GPIO_1V8_5
-Text Label 8600 4700 2    50   ~ 0
+Text Label 8600 3500 2    50   ~ 0
 GPIO_1V8_6
+Text Label 8600 5700 2    50   ~ 0
+GPIO_1V8_7
 Text Label 8600 900  2    50   ~ 0
-GPIO_1V8_7
-Text Label 8600 4400 2    50   ~ 0
 GPIO_1V8_8
-Text Label 8600 3500 2    50   ~ 0
+Text Label 8600 5800 2    50   ~ 0
 GPIO_1V8_9
-Text Label 8600 4600 2    50   ~ 0
+Text Label 8600 4500 2    50   ~ 0
 GPIO_1V8_10
 Text Label 8600 5200 2    50   ~ 0
@@
 Text Label 8600 5400 2    50   ~ 0
 GPIO_1V8_13
+Text Label 8600 4700 2    50   ~ 0
+GPIO_1V8_14
 Text Label 8600 5500 2    50   ~ 0
-GPIO_1V8_14
-Text Label 8600 4500 2    50   ~ 0
 GPIO_1V8_15
-Text Label 8600 5700 2    50   ~ 0
+Text Label 8600 4400 2    50   ~ 0
 GPIO_1V8_16
 Text Label 5050 4850 0    50   ~ 0
@@
 Text Label 5050 6750 0    50   ~ 0
 CLK_1V8_1
-Text Label 8600 5800 2    50   ~ 0
+Text Label 8600 4600 2    50   ~ 0
 GPIO_1V8_17
 Text Label 8600 3400 2    50   ~ 0
