File: pcb/fpga-decoupling.sch (KiCad schematic (older format))
At the start: 0 parts

Commit message: Finished initial schematic. Pin assignments will likely change during routing. Ready for test point insertion and signoff review.
Parts:
- added C100, C101, C102, C103, C104, C105, C63, C64, C65, C66, C67, C68, C69, C70, C77, C83, C85, C86, C89, C90, C91, C92, C93, C94, C95, C96, C97, C98, C99: 0.47 uF, symbol device:C
- added C56: 330 uF, symbol device:C
- added C57, C58, C59, C60, C61, C62, C73, C74, C78, C79, C80, C81, C82, C84, C87, C88: 4.7 uF, symbol device:C
- added C71, C75, C76: 47 uF, symbol device:C
- added C72: 100 uF, symbol device:C
Connections:
- new net 1V0: C56.1, C57.1, C58.1, C59.1, C60.1, C61.1, C62.1, C63.1, C64.1, C65.1, C66.1, C67.1, C68.1, C69.1, C70.1, C77.1, C83.1
- new net 1V8: C100.1, C101.1, C105.1, C71.1, C76.1, C78.1, C82.1, C84.1, C88.1, C89.1, C93.1, C95.1, C96.1
- new net 2V5: C104.1, C75.1, C81.1, C87.1, C92.1, C94.1, C99.1
- new net 3V3: C102.1, C103.1, C72.1, C73.1, C74.1, C79.1, C80.1, C85.1, C86.1, C90.1, C91.1, C97.1, C98.1
- new net GND: C100.2, C101.2, C102.2, C103.2, C104.2, C105.2, C56.2, C57.2, C58.2, C59.2, C60.2, C61.2, C62.2, C63.2, C64.2, C65.2, C66.2, C67.2, C68.2, C69.2, C70.2, C71.2, C72.2, C73.2, C74.2, C75.2, C76.2, C77.2, C78.2, C79.2, C80.2, C81.2, C82.2, C83.2, C84.2, C85.2, C86.2, C87.2, C88.2, C89.2, C90.2, C91.2, C92.2, C93.2, C94.2, C95.2, C96.2, C97.2, C98.2, C99.2
Other:
- note added: "Bank 14"
- note added: "Bank 15"
- note added: "Bank 34"
- note added: "Bank 35"
- note added: "Populate for 7A75T and larger only"
- note added: "Populate for all densities"
- note added: "Populate one cap for 7A50T and smaller, both for 7A75T and larger"
- note added: "Shared by banks 0, 14, 15"
- note added: "VCCAUX:\n* All densities: 3x 0.47, 2x 4.7, 1x 47"
- note added: "VCCBRAM:\n* 7A50T and smaller: 1x 0.47 uF\n* 7A75T and larger: 2x 0.47 uF"
- note added: "VCCINT:\n* 7A100T: 8x 0.47, 6x 4.7\n* 7A50T: 5x 0.47, 3x 4.7\n* Both get a single 330 uF"
- note added: "VCCO, per bank:\n* All densities: 1x 100 uF (can be shared between rails), 2x 4.7 uF, 4x 0.47 uF"
- note added: "VCCO_0:\n* All densities: 1x 47 uF (shared with 100 uF from VCCO_14/15)"

Commit message: Assigned lots of footprints. Still have a few to go.
Parts:
- C100, C101, C102, C103, C104, C105, C63, C64, C65, C66, C67, C68, C69, C70, C77, C83, C85, C86, C89, C90, C91, C92, C93, C94, C95, C96, C97, C98, C99: footprint (none) -> azonenberg_pcb:EIA_0402_CAP_NOSILK
- C56: footprint (none) -> azonenberg_pcb:EIA_1210_CAP_NOSILK
- C57, C58, C59, C60, C61, C62, C73, C74, C78, C79, C80, C81, C82, C84, C87, C88: footprint (none) -> azonenberg_pcb:EIA_0603_CAP_NOSILK
- C71, C72, C75, C76: footprint (none) -> azonenberg_pcb:EIA_1206_CAP_NOSILK
