File: pcb/integralstick.kicad_pcb (KiCad board)
At the start: 4 copper layers, 95 x 59.8 mm, 251 parts, among them J1 CONN_INTEGRALSTICK_FPGA_DEVICE, J2 CONN_INTEGRALSTICK_MCU_DEVICE, Q1 SSM6N58NU, Q2 SSM6N58NU, Q3 SSM6N58NU, U1 STM32F777NIH6‎, U10 DSC6083MI2A-032K768, U12 DSC6001HI2A-025.0000‎, U2 XC7A50T-1FTG256C, U3 S27KS0641, U4 S27KS0641, U5 KSZ9031RN, U6 S25FL064LABNFI011‎, U7 LTC3374-QFN, U8 DSC6001HI2A-025.0000, U9 AT24MAC402-UDFN

Commit message: Finished initial routing
Parts:
- added TP11: TESTPAD, azonenberg_pcb:TESTPOINT_SMT_0.5MM, F.Cu at (90.7, 31.2)
- C10, C118, C15, C16, C18, C19, C22, C23, C3, C45, C73, C74, C79, R20, R36, R38, R41, R43, R44: moved to B.Cu
- moved TP5 61.7 mm to (81.7, 74.3)
- moved R31 61.6 mm to (35.0, 42.5), turned to 90 degrees
- moved TP7 59.8 mm to (75.9, 75.1)
- moved C74 58.7 mm to (75.2, 29.4), turned to 270 degrees
- moved C73 58.3 mm to (70.8, 37.8), turned to 180 degrees
- moved TP6 55.4 mm to (64.5, 61.5)
- moved R33 52.5 mm to (115.8, 28.0), turned to 90 degrees
- moved C79 51.2 mm to (72.5, 54.4)
- moved R36 48.7 mm to (41.0, 70.1), turned to 180 degrees
- moved R41 45.7 mm to (43.9, 70.0), turned to 270 degrees
- moved R38 40.3 mm to (45.9, 69.0), turned to 270 degrees
- moved R43 40.0 mm to (46.8, 67.5), turned to 180 degrees
- moved C118 31.5 mm to (94.7, 58.1), turned to 45 degrees
- moved C16 29.3 mm to (94.3, 53.7), turned to 90 degrees
- moved C15 29.0 mm to (88.3, 50.8), turned to 180 degrees
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Connections:
- J2 pad 10: /FPGA_RST_N -> /Ethernet/ETH_B_P
- J2 pad 109: /GND -> /3V3
- J2 pad 11: /FPGA_DONE -> Net-(J2-Pad11)
- J2 pad 110: /GND -> /3V3
- J2 pad 111: /Ethernet/ETH_D_N -> Net-(J2-Pad111)
- J2 pad 112: /Ethernet/ETH_C_N -> Net-(J2-Pad112)
- J2 pad 113: /Ethernet/ETH_D_P -> /MCU_RST_N
- J2 pad 114: /Ethernet/ETH_C_P -> Net-(J2-Pad114)
- J2 pad 115: /GND -> /3V3
- J2 pad 116: /GND -> /3V3
- J2 pad 117: /Ethernet/ETH_B_N -> Net-(J2-Pad117)
- J2 pad 118: /JTAG_TMS -> Net-(J2-Pad118)
- J2 pad 119: /Ethernet/ETH_B_P -> Net-(J2-Pad119)
- J2 pad 12: /MCU_BOOT0 -> /Ethernet/ETH_B_N
- J2 pad 120: /MCU_TDO -> /FPGA_DONE
- J2 pad 14: /3V3 -> /GND
- J2 pad 16: Net-(J2-Pad16) -> /Ethernet/ETH_C_P
- J2 pad 18: Net-(J2-Pad18) -> /Ethernet/ETH_C_N
- J2 pad 2: /3V3 -> /GND
- J2 pad 20: /3V3 -> /GND
- J2 pad 22: Net-(J2-Pad22) -> /Ethernet/ETH_D_P
- J2 pad 24: Net-(J2-Pad24) -> /Ethernet/ETH_D_N
- J2 pad 26: /3V3 -> /GND
- J2 pad 3: /FPGA_TDI -> Net-(J2-Pad3)
- J2 pad 5: /JTAG_TCK -> Net-(J2-Pad5)
- J2 pad 64: Net-(J2-Pad64) -> /JTAG_TCK
- J2 pad 66: Net-(J2-Pad66) -> /FPGA_TDI
- J2 pad 70: Net-(J2-Pad70) -> /JTAG_TMS
- J2 pad 72: Net-(J2-Pad72) -> /MCU_TDO
- J2 pad 76: Net-(J2-Pad76) -> /FPGA_RST_N
- J2 pad 78: Net-(J2-Pad78) -> /MCU_BOOT0
- J2 pad 8: /3V3 -> /GND
- J2 pad 9: /MCU_RST_N -> Net-(J2-Pad9)
- U1 pad A1: Net-(J2-Pad77) -> Net-(J2-Pad93)
- U1 pad A11: Net-(J2-Pad58) -> Net-(J2-Pad60)
- U1 pad A12: Net-(J2-Pad45) -> Net-(J2-Pad52)
- U1 pad A2: Net-(J2-Pad76) -> Net-(J2-Pad87)
- U1 pad A3: Net-(J2-Pad75) -> Net-(J2-Pad83)
- U1 pad A5: Net-(J2-Pad72) -> Net-(J2-Pad81)
- U1 pad A6: Net-(J2-Pad71) -> Net-(J2-Pad77)
- U1 pad A8: Net-(J2-Pad33) -> Net-(J2-Pad75)
- U1 pad A9: Net-(J2-Pad30) -> Net-(J2-Pad71)
- U1 pad B1: Net-(J2-Pad78) -> Net-(J2-Pad95)
- U1 pad B11: Net-(J2-Pad57) -> Net-(J2-Pad58)
- U1 pad B12: Net-(J2-Pad47) -> Net-(J2-Pad54)
- U1 pad B15: Net-(J2-Pad24) -> Net-(J2-Pad40)
- U1 pad B2: Net-(J2-Pad81) -> Net-(J2-Pad89)
- U1 pad C10: Net-(J2-Pad54) -> Net-(J2-Pad69)
- U1 pad C11: Net-(J2-Pad52) -> Net-(J2-Pad63)
- U1 pad C15: Net-(J2-Pad23) -> Net-(J2-Pad36)
- U1 pad D1: Net-(J2-Pad46) -> Net-(J2-Pad99)
- U1 pad D11: Net-(J2-Pad53) -> Net-(J2-Pad65)
- U1 pad D12: Net-(J2-Pad51) -> Net-(J2-Pad46)
- U1 pad D15: Net-(J2-Pad22) -> Net-(J2-Pad34)
- U1 pad D2: Net-(J2-Pad95) -> Net-(J2-Pad101)
- U1 pad E15: Net-(J2-Pad21) -> Net-(J2-Pad30)
- U1 pad E2: Net-(J2-Pad96) -> Net-(J2-Pad105)
- U1 pad F15: Net-(J2-Pad18) -> Net-(J2-Pad28)
- U1 pad G2: Net-(J2-Pad99) -> Net-(J2-Pad107)
- U1 pad H2: Net-(J2-Pad100) -> Net-(J2-Pad111)
- U1 pad J2: Net-(J2-Pad101) -> Net-(J2-Pad117)
- U1 pad K1: Net-(J2-Pad106) -> Net-(J2-Pad90)
- U1 pad K13: Net-(J2-Pad70) -> Net-(J2-Pad57)
- U1 pad K15: Net-(J2-Pad63) -> Net-(J2-Pad59)
- U1 pad K2: Net-(J2-Pad105) -> Net-(J2-Pad94)
- U1 pad K3: Net-(J2-Pad102) -> Net-(J2-Pad119)
- U1 pad L12: Net-(J2-Pad69) -> Net-(J2-Pad47)
- U1 pad L14: Net-(J2-Pad60) -> Net-(J2-Pad53)
- U1 pad L15: Net-(J2-Pad59) -> Net-(J2-Pad51)
- U1 pad L2: Net-(J2-Pad108) -> Net-(J2-Pad100)
- U1 pad L3: Net-(J2-Pad107) -> Net-(J2-Pad96)
- U1 pad L4: Net-(J2-Pad41) -> Net-(J2-Pad102)
- U1 pad M10: Net-(J2-Pad65) -> Net-(J2-Pad23)
- U1 pad M11: Net-(J2-Pad66) -> Net-(J2-Pad33)
- U1 pad M2: Net-(J2-Pad39) -> Net-(J2-Pad112)
- U1 pad M4: Net-(J2-Pad40) -> Net-(J2-Pad88)
- U1 pad M5: Net-(J2-Pad29) -> Net-(J2-Pad84)
- U1 pad N10: Net-(J2-Pad64) -> Net-(J2-Pad21)
- U1 pad N3: Net-(J2-Pad15) -> Net-(J2-Pad108)
- U1 pad N9: Net-(J2-Pad83) -> Net-(J2-Pad5)
- U1 pad P10: Net-(J2-Pad88) -> Net-(J2-Pad15)
- U1 pad P11: Net-(J2-Pad93) -> Net-(J2-Pad29)
- U1 pad P12: Net-(J2-Pad34) -> Net-(J2-Pad39)
- U1 pad P4: Net-(J2-Pad17) -> Net-(J2-Pad114)
- U1 pad P9: Net-(J2-Pad84) -> Net-(J2-Pad11)
- U1 pad R10: Net-(J2-Pad89) -> Net-(J2-Pad17)
- U1 pad R11: Net-(J2-Pad94) -> Net-(J2-Pad27)
- U1 pad R12: Net-(J2-Pad90) -> Net-(J2-Pad35)
- U1 pad R14: Net-(J2-Pad35) -> Net-(J2-Pad45)
- U1 pad R15: Net-(J2-Pad36) -> Net-(J2-Pad41)
- U1 pad R2: Net-(J2-Pad16) -> Net-(J2-Pad106)
- U1 pad R4: Net-(J2-Pad28) -> Net-(J2-Pad118)
- U1 pad R5: Net-(J2-Pad27) -> Net-(J2-Pad82)
- U1 pad R8: Net-(J2-Pad82) -> Net-(J2-Pad3)
- U1 pad R9: Net-(J2-Pad87) -> Net-(J2-Pad9)
- U2 pad L13: /MCU/RMII_RXD0 -> /MCU/UART6_RX
- U2 pad L14: /MCU/RMII_CRS_DV -> /MCU/DCMI_PIXCLK
- U2 pad M12: /MCU/RMII_TXD0 -> /MCU/SPI5_MOSI
- U2 pad M14: /MCU/RMII_RXD1 -> /MCU/DCMI_D7
- U2 pad M16: /MCU/RMII_TXD1 -> /MCU/SPI5_SCK
- U2 pad M6: /MCU/DCMI_D7 -> /MCU/DCMI_D6
- U2 pad N12: /MCU/SPI5_SCK -> /MCU/DCMI_D4
- U2 pad N13: /MCU/DCMI_D0 -> Net-(R22-Pad1)
- U2 pad N14: /MCU/SPI5_MOSI -> /MCU/RMII_MDC
- U2 pad N16: /MCU/RMII_MDC -> /MCU/SPI5_CS_N
- U2 pad N9: /MCU/SPI5_MISO -> /MCU/UART6_TX
- U2 pad P10: /MCU/DCMI_D4 -> /MCU/SPI5_MISO
- U2 pad P14: /MCU/DCMI_PIXCLK -> /MCU/RMII_CRS_DV
- U2 pad P15: /MCU/DCMI_D1 -> /MCU/RMII_TXD0
- U2 pad P16: /MCU/DCMI_D3 -> /MCU/DCMI_HSYNC
- U2 pad R12: /MCU/DCMI_HSYNC -> /MCU/DCMI_D5
- U2 pad R13: /MCU/UART6_RX -> /MCU/DCMI_D1
- U2 pad R15: /MCU/DCMI_VSYNC -> /MCU/RMII_RXD1
- U2 pad R16: Net-(R22-Pad1) -> /MCU/RMII_RXD0
- U2 pad T12: /MCU/SPI5_CS_N -> /MCU/DCMI_VSYNC
- U2 pad T13: /MCU/UART6_TX -> /MCU/DCMI_D3
- U2 pad T14: /MCU/DCMI_D6 -> /MCU/DCMI_D0
- U2 pad T15: /MCU/DCMI_D5 -> /MCU/RMII_TXD1
Routing:
- net /3V3: track 393.5 -> 576.0 mm, vias 92 -> 138
- net /GND: track 821.5 -> 1003.1 mm, vias 228 -> 263
- net /Power Supply/3V3_SENSE: track 0.00 -> 122.6 mm, vias 0 -> 1
- net /PSU_TEMP: track 57.1 -> 136.1 mm, vias 4 -> 9
- net /FPGA_RST_N: track 25.4 -> 79.5 mm, vias 1 -> 3
- net Net-(J2-Pad3): track 0.00 -> 53.7 mm, vias 0 -> 1
- net Net-(J2-Pad5): track 0.00 -> 53.2 mm, vias 0 -> 1
- net /FPGA_TDI: track 24.5 -> 77.6 mm, vias 1 -> 4
- net /JTAG_TCK: track 32.8 -> 85.6 mm, vias 2 -> 4
- net /JTAG_TMS: track 28.8 -> 81.4 mm, vias 2 -> 4
- net Net-(J2-Pad9): track 0.00 -> 51.8 mm, vias 0 -> 1
- net Net-(J2-Pad11): track 0.00 -> 49.0 mm, vias 0 -> 1
- net Net-(J2-Pad17): track 0.00 -> 47.0 mm, vias 0 -> 1
- net Net-(J2-Pad29): track 0.00 -> 44.8 mm, vias 0 -> 1
- net Net-(J2-Pad27): track 0.00 -> 44.7 mm, vias 0 -> 1
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- added copper zone on In1.Cu, net /GND
Other:
- board size 95 x 59.8 mm -> 87 x 59.8 mm
- board text added: "1V0"
- board text added: "1V2"
- board text added: "GND"
- board text added: "VBAT"
