File: pcb/psu.sch (KiCad schematic (older format))
At the start: 47 parts, among them J1 CONN_INTEGRALSTICK_FPGA_DEVICE, J2 CONN_INTEGRALSTICK_MCU_DEVICE, U1 STM32F777NIH6‎, U2 XC7A50T-1FTG256C, U7 LTC3374-QFN

Commit message: Updated integralstick schematic to fix library paths. No content changes.
Parts:
- TP11, TP2, TP3: symbol conn:CONN_01X01 -> integralstick-rescue:CONN_01X01-conn
Changed lines of the file:
@@
 AR Path="/5B6B703A/5B8A9FBF" Ref="J?"  Part="2"
 AR Path="/5B6B7005/5B8A9FBF" Ref="J1"  Part="1"
+AR Path="/5B8A9FBF" Ref="J1"  Part="1"
 F 0 "J1" H 4500 10750 50  0000 C CNN
 F 1 "CONN_INTEGRALSTICK_FPGA_DEVICE" H 4700 10850 50  0000 C CNN
@@
 3V3
 $Comp
-L conn:CONN_01X01 TP2
+L integralstick-rescue:CONN_01X01-conn TP2
 U 1 1 5C1887D2
 P 5050 6450
+AR Path="/5C1887D2" Ref="TP2"  Part="1"
+AR Path="/5B6B7005/5C1887D2" Ref="TP2"  Part="1"
 F 0 "TP2" H 5128 6491 50  0000 L CNN
 F 1 "TESTPAD" H 5128 6400 50  0000 L CNN
@@
 	4150 6350 4000 6350
 $Comp
-L conn:CONN_01X01 TP3
+L integralstick-rescue:CONN_01X01-conn TP3
 U 1 1 5C1FEFFC
 P 5050 6750
+AR Path="/5C1FEFFC" Ref="TP3"  Part="1"
+AR Path="/5B6B7005/5C1FEFFC" Ref="TP3"  Part="1"
 F 0 "TP3" H 5128 6791 50  0000 L CNN
 F 1 "TESTPAD" H 5128 6700 50  0000 L CNN
@@
 	4150 8350 4150 8450
 $Comp
-L conn:CONN_01X01 TP?
+L integralstick-rescue:CONN_01X01-conn TP?
 U 1 1 5C11F6A8
 P 8650 6550
