File: host-full/mcu.sch (KiCad schematic (older format))
At the start: 9 parts, among them J1 CONN_INTEGRALSTICK_MCU_HOST, J10 PMOD_HOST, J11 PMOD_HOST, J12 PMOD_HOST, J13 PMOD_HOST, J14 PMOD_HOST, J7 PMOD_HOST, J8 PMOD_HOST, J9 PMOD_HOST

Commit message: Initial layout on host-full. Rough floorplan is finalized, all MCU PMODs routed.
Parts:
- J1: footprint (none) -> azonenberg_pcb:CONN_SAMTEC_QSH-060-01-L-D-A
- J10, J11, J12, J13, J14, J7, J8, J9: footprint (none) -> azonenberg_pcb:CONN_HEADER_2.54MM_2x6_RA_PMOD_HOST
Connections:
- net PA0: now also J8.10 (D7); no longer J7.7 (D4)
- net PA10: now also J12.3 (D2); no longer J7.3 (D2)
- net PA11: now also J12.1 (D0); no longer J7.1 (D0)
- net PA12: now also J12.4 (D3); no longer J7.4 (D3)
- net PA3: now also J8.4 (D3); no longer J7.8 (D5)
- net PA5: now also J9.1 (D0); no longer J7.9 (D6)
- net PA8: now also J7.1 (D0); no longer J7.10 (D7)
- net PA9: now also J12.2 (D1); no longer J7.2 (D1)
- net PB0: now also J12.9 (D6); no longer J8.1 (D0)
- net PB1: now also J9.2 (D1); no longer J8.2 (D1)
- net PB10: now also J11.2 (D1); no longer J8.8 (D5)
- net PB14: now also J11.1 (D0); no longer J8.9 (D6)
- net PB15: now also J11.8 (D5); no longer J8.10 (D7)
- net PB2: now also J12.10 (D7); no longer J8.3 (D2)
- net PB4: now also J13.7 (D4); no longer J8.4 (D3)
- net PB5: now also J10.10 (D7); no longer J8.7 (D4)
- net PC0: now also J9.7 (D4); no longer J14.1 (D0)
- net PC10: now also J7.2 (D1); no longer J14.4 (D3)
- net PC12: now also J7.4 (D3); no longer J14.7 (D4)
- net PC13: now also J9.10 (D7); no longer J14.8 (D5)
- net PC2: now also J8.1 (D0); no longer J14.2 (D1)
- net PC3: now also J8.9 (D6); no longer J14.3 (D2)
- net PD0: now also J7.10 (D7); no longer J12.1 (D0)
- net PD1: now also J7.9 (D6); no longer J12.2 (D1)
- net PD10: now also J13.9 (D6); no longer J13.3 (D2)
- net PD11: now also J14.1 (D0); no longer J13.4 (D3)
- net PD12: now also J14.7 (D4); no longer J13.7 (D4)
- net PD13: now also J11.3 (D2); no longer J13.8 (D5)
- net PD14: now also J11.7 (D4); no longer J13.9 (D6)
- net PD15: now also J13.3 (D2); no longer J13.10 (D7)
- net PD2: now also J7.3 (D2); no longer J12.3 (D2)
- net PD3: now also J13.2 (D1); no longer J12.4 (D3)
- net PD4: now also J13.8 (D5); no longer J12.7 (D4)
- net PD5: now also J13.1 (D0); no longer J12.8 (D5)
- net PD6: now also J12.7 (D4); no longer J12.9 (D6)
- net PD7: now also J12.8 (D5); no longer J12.10 (D7)
- net PD8: now also J13.4 (D3); no longer J13.1 (D0)
- net PD9: now also J13.10 (D7); no longer J13.2 (D1)
- net PE0: now also J10.4 (D3); no longer J10.1 (D0)
- net PE1: now also J10.9 (D6); no longer J10.2 (D1)
- net PE10: now also J14.3 (D2); no longer J11.3 (D2)
- net PE11: now also J14.2 (D1); no longer J11.4 (D3)
- net PE12: now also J14.8 (D5); no longer J11.7 (D4)
- net PE13: now also J11.9 (D6); no longer J11.8 (D5)
- net PE14: now also J11.10 (D7); no longer J11.9 (D6)
- net PE15: now also J11.4 (D3); no longer J11.10 (D7)
- net PE3: now also J10.8 (D5); no longer J10.4 (D3)
- net PE5: now also J10.1 (D0); no longer J10.8 (D5)
- net PE6: now also J10.2 (D1); no longer J10.9 (D6)
- net PE7: now also J14.4 (D3); no longer J10.10 (D7)
- net PE8: now also J14.10 (D7); no longer J11.1 (D0)
- net PE9: now also J14.9 (D6); no longer J11.2 (D1)
- net PF0: now also J9.4 (D3); no longer J9.1 (D0)
- net PF1: now also J9.9 (D6); no longer J9.2 (D1)
- net PF3: now also J9.8 (D5); no longer J9.4 (D3)
- net PF6: now also J8.2 (D1); no longer J9.7 (D4)
- net PF7: now also J8.7 (D4); no longer J9.8 (D5)
- net PF8: now also J8.8 (D5); no longer J9.9 (D6)
- net PF9: now also J8.3 (D2); no longer J9.10 (D7)
- no-connect marks 4 -> 3
Other:
- moved on the sheet: J11, J12, J13, J14, J1D, J1E, J1F, J1I, J7, J8
