File: host-full/psu.sch (KiCad schematic (older format))
At the start: 6 parts, among them J1 CONN_INTEGRALSTICK_MCU_HOST, J2 CONN_INTEGRALSTICK_FPGA_HOST, K1 CONN_3_PWROUT

Commit message: Finished initial schematic review
Parts:
- added C85: 0.1 uF, symbol device:C
- added C86: 4.7 nF, symbol device:C
- added C87: 22 uF, symbol device:C
- added C88: 47 uF, symbol device:C
- added J22, J24, J25, J26, J27, J28: TESTPAD, symbol Connector:Conn_01x01
- added J29, J30, J31: TESTCLIP, symbol Connector:Conn_01x01
- added L11: 1 uH, symbol passive-azonenberg:INDUCTOR_PWROUT
- added R53: 10K, symbol device:R
- added R54: 1, symbol device:R
- added U7: SC185EUL, symbol power-azonenberg:SC185
Connections:
- net 1V8: now also J25.1 (Pin_1)
- net 2V5: now also J26.1 (Pin_1)
- net 3V3: now also J27.1 (Pin_1)
- net 5V0: now also C87.2, J28.1 (Pin_1), R53.1, R54.1, U7.1 (PVIN), U7.2 (PVIN), U7.5 (MODE), U7.6 (EN)
- net GND: now also C85.1, C86.2, C87.1, C88.2, J29.1 (Pin_1), J30.1 (Pin_1), J31.1 (Pin_1), U7.11 (PGND), U7.12 (PGND), U7.13 (PGND), U7.3 (AGND), U7.PAD
- new net: L11.2, U7.14 (LX), U7.15 (LX), U7.16 (LX)
- new net: C85.2, R54.2, U7.4 (AVIN)
- new net: C86.1, U7.9 (SS)
- new net 1V2: C88.1, J24.1 (Pin_1), L11.1, U7.10 (VOUT)
- new net 1V2_PGOOD: J22.1 (Pin_1), R53.2, U7.7 (PGOOD)
Other:
- note added: "1 uH TBD"
- note added: "Power rails:\n3 PHYs * 221 mA = 663 mA @ 1V2\n3 PHYs * 58.8 mA = 176 mA @ 2V5"

Commit message: Initial layout on host-full. Rough floorplan is finalized, all MCU PMODs routed.
Parts:
- C75, C87, C88: footprint (none) -> azonenberg_pcb:EIA_1210_CAP_NOSILK
- C85: footprint (none) -> azonenberg_pcb:EIA_0402_CAP_NOSILK
- C86: footprint (none) -> azonenberg_pcb:EIA_0603_CAP_NOSILK
- F1: footprint (none) -> azonenberg_pcb:EIA_0603_RES_NOSILK
- J1, J2: footprint (none) -> azonenberg_pcb:CONN_SAMTEC_QSH-060-01-L-D-A
- J22, J24, J25, J26, J27, J28: footprint (none) -> azonenberg_pcb:TESTPOINT_SMT_0.5MM
- J29, J30, J31: footprint (none) -> azonenberg_pcb:TESTPOINT_SMT_KEYSTONE_5016
- K1: footprint (none) -> azonenberg_pcb:CONN_CUI_PJ-058BH_HIPWR_BARREL_NOSLOT
- L11: value 1 uH -> NRS5030T1R0NMGJ; footprint (none) -> azonenberg_pcb:EIA_0402_RES_NOSILK
- L7: footprint (none) -> azonenberg_pcb:EIA_1206_CAP_NOSILK
- R53, R54: footprint (none) -> azonenberg_pcb:EIA_0402_RES_NOSILK
- U7: footprint (none) -> azonenberg_pcb:QFN_16_0.5MM_3x3MM
Other:
- note removed: "1 uH TBD"
Changed lines of the file:
@@
 Sheet 2 4
 Title "INTEGRALSTICK Full Host"
-Date "2019-11-04"
+Date "2019-11-07"
 Rev "0.1"
 Comp "Antikernel Labs"
@@
 F 0 "J2" H 13425 11325 50  0000 C CNN
 F 1 "CONN_INTEGRALSTICK_FPGA_HOST" H 13425 11234 50  0000 C CNN
-F 2 "" H 12950 8150 50  0001 C CNN
+F 2 "azonenberg_pcb:CONN_SAMTEC_QSH-060-01-L-D-A" H 12950 8150 50  0001 C CNN
 F 3 "" H 12950 8150 50  0001 C CNN
 	1    12950 8150
@@
 F 0 "J1" H 13450 8425 50  0000 C CNN
 F 1 "CONN_INTEGRALSTICK_MCU_HOST" H 13450 8334 50  0000 C CNN
-F 2 "" H 13000 4650 50  0001 C CNN
+F 2 "azonenberg_pcb:CONN_SAMTEC_QSH-060-01-L-D-A" H 13000 4650 50  0001 C CNN
 F 3 "" H 13000 4650 50  0001 C CNN
 	1    13000 4650
@@
 F 0 "K1" H 1017 1300 50  0000 C CNN
 F 1 "CONN_3_PWROUT" H 1017 1216 40  0000 C CNN
-F 2 "" H 1150 1000 60  0000 C CNN
+F 2 "azonenberg_pcb:CONN_CUI_PJ-058BH_HIPWR_BARREL_NOSLOT" H 1150 1000 60  0001 C CNN
 F 3 "" H 1150 1000 60  0000 C CNN
 	1    1150 1000
@@
 F 0 "F1" H 2350 1140 50  0000 C CNN
 F 1 "2A" H 2350 1049 50  0000 C CNN
-F 2 "" H 2350 900 60  0000 C CNN
+F 2 "azonenberg_pcb:EIA_0603_RES_NOSILK" H 2350 900 60  0001 C CNN
 F 3 "" H 2350 900 60  0000 C CNN
 	1    2350 900
@@
 F 0 "L7" V 2892 900 40  0000 C CNN
 F 1 "BLM31KN271SH1L" V 2968 900 40  0000 C CNN
-F 2 "" H 3050 900 60  0000 C CNN
+F 2 "azonenberg_pcb:EIA_1206_CAP_NOSILK" H 3050 900 60  0001 C CNN
 F 3 "" H 3050 900 60  0000 C CNN
 	1    3050 900
@@
 F 0 "C75" H 3565 1096 50  0000 L CNN
 F 1 "47 uF" H 3565 1005 50  0000 L CNN
-F 2 "" H 3488 900 50  0001 C CNN
+F 2 "azonenberg_pcb:EIA_1210_CAP_NOSILK" H 3488 900 50  0001 C CNN
 F 3 "" H 3450 1050 50  0001 C CNN
 	1    3450 1050
@@
 F 0 "U7" H 3375 4687 60  0000 C CNN
 F 1 "SC185EUL" H 3375 4581 60  0000 C CNN
-F 2 "" H 3400 3600 60  0000 C CNN
+F 2 "azonenberg_pcb:QFN_16_0.5MM_3x3MM" H 3400 3600 60  0001 C CNN
 F 3 "" H 3400 3600 60  0000 C CNN
 	1    3400 3600
@@
 P 4750 2900
 F 0 "L11" V 4592 2900 40  0000 C CNN
-F 1 "1 uH" V 4668 2900 40  0000 C CNN
-F 2 "" H 4750 2900 60  0000 C CNN
+F 1 "NRS5030T1R0NMGJ" V 4668 2900 40  0000 C CNN
+F 2 "azonenberg_pcb:EIA_0402_RES_NOSILK" H 4750 2900 60  0001 C CNN
 F 3 "" H 4750 2900 60  0000 C CNN
 	1    4750 2900
@@
 Wire Wire Line
 	5050 2900 5150 2900
-Text Notes 4900 2550 0    50   ~ 0
-1 uH TBD
 Wire Wire Line
 	4250 2900 4250 3000
@@
 F 0 "R54" H 2370 2996 50  0000 L CNN
 F 1 "1" H 2370 2905 50  0000 L CNN
-F 2 "" V 2230 2950 50  0001 C CNN
+F 2 "azonenberg_pcb:EIA_0402_RES_NOSILK" V 2230 2950 50  0001 C CNN
 F 3 "" H 2300 2950 50  0001 C CNN
 	1    2300 2950
@@
 F 0 "C85" H 1915 2996 50  0000 L CNN
 F 1 "0.1 uF" H 1915 2905 50  0000 L CNN
-F 2 "" H 1838 2800 50  0001 C CNN
+F 2 "azonenberg_pcb:EIA_0402_CAP_NOSILK" H 1838 2800 50  0001 C CNN
 F 3 "" H 1800 2950 50  0001 C CNN
 	1    1800 2950
@@
 F 0 "C86" H 1915 3696 50  0000 L CNN
 F 1 "4.7 nF" H 1915 3605 50  0000 L CNN
-F 2 "" H 1838 3500 50  0001 C CNN
+F 2 "azonenberg_pcb:EIA_0603_CAP_NOSILK" H 1838 3500 50  0001 C CNN
 F 3 "" H 1800 3650 50  0001 C CNN
 	1    1800 3650
@@
 F 0 "J22" H 1168 3175 50  0000 C CNN
 F 1 "TESTPAD" H 1168 3266 50  0000 C CNN
-F 2 "" H 1250 3400 50  0001 C CNN
+F 2 "azonenberg_pcb:TESTPOINT_SMT_0.5MM" H 1250 3400 50  0001 C CNN
 F 3 "~" H 1250 3400 50  0001 C CNN
 	1    1250 3400
@@
 F 0 "R53" H 1670 3296 50  0000 L CNN
 F 1 "10K" H 1670 3205 50  0000 L CNN
-F 2 "" V 1530 3250 50  0001 C CNN
+F 2 "azonenberg_pcb:EIA_0402_RES_NOSILK" V 1530 3250 50  0001 C CNN
 F 3 "" H 1600 3250 50  0001 C CNN
 	1    1600 3250
@@
 F 0 "C87" H 2415 2696 50  0000 L CNN
 F 1 "22 uF" H 2415 2605 50  0000 L CNN
-F 2 "" H 2338 2500 50  0001 C CNN
+F 2 "azonenberg_pcb:EIA_1210_CAP_NOSILK" H 2338 2500 50  0001 C CNN
 F 3 "" H 2300 2650 50  0001 C CNN
 	1    2300 2650
@@
 F 0 "C88" H 5165 3096 50  0000 L CNN
 F 1 "47 uF" H 5165 3005 50  0000 L CNN
-F 2 "" H 5088 2900 50  0001 C CNN
+F 2 "azonenberg_pcb:EIA_1210_CAP_NOSILK" H 5088 2900 50  0001 C CNN
 F 3 "" H 5050 3050 50  0001 C CNN
 	1    5050 3050
@@
 F 0 "J24" H 1168 4275 50  0000 C CNN
 F 1 "TESTPAD" H 1168 4366 50  0000 C CNN
-F 2 "" H 1250 4500 50  0001 C CNN
+F 2 "azonenberg_pcb:TESTPOINT_SMT_0.5MM" H 1250 4500 50  0001 C CNN
 F 3 "~" H 1250 4500 50  0001 C CNN
 	1    1250 4500
@@
 F 0 "J25" H 1168 4675 50  0000 C CNN
 F 1 "TESTPAD" H 1168 4766 50  0000 C CNN
-F 2 "" H 1250 4900 50  0001 C CNN
+F 2 "azonenberg_pcb:TESTPOINT_SMT_0.5MM" H 1250 4900 50  0001 C CNN
 F 3 "~" H 1250 4900 50  0001 C CNN
 	1    1250 4900
@@
 F 0 "J26" H 1168 5025 50  0000 C CNN
 F 1 "TESTPAD" H 1168 5116 50  0000 C CNN
-F 2 "" H 1250 5250 50  0001 C CNN
+F 2 "azonenberg_pcb:TESTPOINT_SMT_0.5MM" H 1250 5250 50  0001 C CNN
 F 3 "~" H 1250 5250 50  0001 C CNN
 	1    1250 5250
@@
 F 0 "J27" H 1168 5375 50  0000 C CNN
 F 1 "TESTPAD" H 1168 5466 50  0000 C CNN
-F 2 "" H 1250 5600 50  0001 C CNN
+F 2 "azonenberg_pcb:TESTPOINT_SMT_0.5MM" H 1250 5600 50  0001 C CNN
 F 3 "~" H 1250 5600 50  0001 C CNN
 	1    1250 5600
@@
 F 0 "J28" H 1168 5725 50  0000 C CNN
 F 1 "TESTPAD" H 1168 5816 50  0000 C CNN
-F 2 "" H 1250 5950 50  0001 C CNN
+F 2 "azonenberg_pcb:TESTPOINT_SMT_0.5MM" H 1250 5950 50  0001 C CNN
 F 3 "~" H 1250 5950 50  0001 C CNN
 	1    1250 5950
@@
 F 0 "J29" H 1168 6075 50  0000 C CNN
 F 1 "TESTCLIP" H 1168 6166 50  0000 C CNN
-F 2 "" H 1250 6300 50  0001 C CNN
+F 2 "azonenberg_pcb:TESTPOINT_SMT_KEYSTONE_5016" H 1250 6300 50  0001 C CNN
 F 3 "~" H 1250 6300 50  0001 C CNN
 	1    1250 6300
@@
 F 0 "J30" H 1168 6425 50  0000 C CNN
 F 1 "TESTCLIP" H 1168 6516 50  0000 C CNN
-F 2 "" H 1250 6650 50  0001 C CNN
+F 2 "azonenberg_pcb:TESTPOINT_SMT_KEYSTONE_5016" H 1250 6650 50  0001 C CNN
 F 3 "~" H 1250 6650 50  0001 C CNN
 	1    1250 6650
@@
 F 0 "J31" H 1168 6775 50  0000 C CNN
 F 1 "TESTCLIP" H 1168 6866 50  0000 C CNN
-F 2 "" H 1250 7000 50  0001 C CNN
+F 2 "azonenberg_pcb:TESTPOINT_SMT_KEYSTONE_5016" H 1250 7000 50  0001 C CNN
 F 3 "~" H 1250 7000 50  0001 C CNN
 	1    1250 7000

Commit message: Finished initial routing, still need to do planes and design review
Parts:
- L11: footprint azonenberg_pcb:EIA_0402_RES_NOSILK -> azonenberg_pcb:INDUCTOR_YUDEN_NRS5030
Changed lines of the file:
@@
 F 0 "L11" V 4592 2900 40  0000 C CNN
 F 1 "NRS5030T1R0NMGJ" V 4668 2900 40  0000 C CNN
-F 2 "azonenberg_pcb:EIA_0402_RES_NOSILK" H 4750 2900 60  0001 C CNN
+F 2 "azonenberg_pcb:INDUCTOR_YUDEN_NRS5030" H 4750 2900 60  0001 C CNN
 F 3 "" H 4750 2900 60  0000 C CNN
 	1    4750 2900
